File: PCB_Capteur/PCB_Capteur.kicad_sch (KiCad schematic)
At the start: 15 parts, among them J1 Conn_01x08_Socket, J2 Conn_ESP32_Custom, J3 Conn_01x02_Socket, U1 DM-OLED096-636

Commit message: Adding Images for the readme
Connections:
- net GND: no longer LTC1050.5 (CLK)
- no-connect marks 22 -> 23
Changed lines of the file:
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@@
-	)
-	(junction
-		(at 90.17 63.5)
-		(diameter 0)
-		(color 0 0 0 0)
 	)
 	(junction
@@
 	)
 	(no_connect
+		(at 90.17 53.34)
+	)
+	(no_connect
 		(at 233.68 99.06)
 	)
@@
 	(wire
 		(pts
-			(xy 73.66 63.5) (xy 90.17 63.5)
+			(xy 73.66 63.5) (xy 123.19 63.5)
 		)
 		(stroke
@@
 	(wire
 		(pts
-			(xy 90.17 53.34) (xy 90.17 63.5)
-		)
-		(stroke
-			(width 0)
-			(type default)
-		)
-	)
-	(wire
-		(pts
 			(xy 229.87 81.28) (xy 233.68 81.28)
 		)
 		(stroke
-			(width 0)
-			(type default)
-		)
-	)
-	(wire
-		(pts
-			(xy 90.17 63.5) (xy 123.19 63.5)
-		)
-		(stroke
